File: sous-vide_controller/sous-vide_controller.sch (KiCad schematic (older format))
At the start: 0 parts

Commit message: first draft of controller hookup schematic
Parts:
- added J1: NEIGHBOR2, gsg-modules:HEADER-2x20, symbol sous-vide_controller-rescue:CONN_02X20-
- added J2: NEIGHBOR1, gsg-modules:HEADER-2x20, symbol sous-vide_controller-rescue:CONN_02X20-
- added LCD1: ADM1602K, symbol gsg-symbols:ADM1602K
- added U1, U2: IoT_Relay, symbol gsg-symbols:IoT_Relay
- added U3: DS18B20, Package_TO_SOT_THT:TO-92_Inline, symbol Sensor_Temperature:DS18B20
Connections:
- net labels added: ADC0_0, CLK0, CLK2, GND, I2C0_SCL, I2C0_SDA, P0_0, P0_1, P1_0, P1_1, P1_10, P1_11, P1_12, P1_13, P1_14, P1_15, P1_16, P1_17, P1_18, P1_19, P1_2, P1_20, P1_3, P1_4, P1_5, P1_6, P1_7, P1_8, P1_9, P2_0, P2_1, P2_2, P2_3, P2_4, P2_5, P2_6, P2_7, P2_8, P3_0, P3_1, P3_2, P3_3, P3_4, P3_5, P3_6, P3_7, P4_0, P4_10, P4_2, P4_3, P4_4, P4_5, P4_6, P4_7, P4_8, P4_9, P5_0, P5_1, P5_2, P5_3, P5_4, P5_5, P5_6, P5_7, P6_0, P6_3, P6_6, P6_7, P6_8, P7_0, P7_1, P7_2, P7_7, P9_5, P9_6, PF_4, VBUS, VCC, WAKEUP0
- wire segments 0 -> 96
Other:
- note added: "BOOT"
- note added: "DFU"
- note added: "ISP"
- note added: "MISO"
- note added: "MOSI"
- note added: "SCK"
- note added: "SSEL"

Commit message: added resistor to controller hook-up schematic
Parts:
- added R1: 4.7k, symbol Device:R
Connections:
- wire segments 96 -> 103
Other:
- moved on the sheet: U3
Changed lines of the file:
@@
 L Sensor_Temperature:DS18B20 U3
 U 1 1 5BE9875D
-P 4850 2700
-F 0 "U3" H 4620 2746 50  0000 R CNN
-F 1 "DS18B20" H 4620 2655 50  0000 R CNN
-F 2 "Package_TO_SOT_THT:TO-92_Inline" H 3850 2450 50  0001 C CNN
-F 3 "http://datasheets.maximintegrated.com/en/ds/DS18B20.pdf" H 4700 2950 50  0001 C CNN
-	1    4850 2700
+P 6150 1850
+F 0 "U3" H 5920 1896 50  0000 R CNN
+F 1 "DS18B20" H 5920 1805 50  0000 R CNN
+F 2 "Package_TO_SOT_THT:TO-92_Inline" H 5150 1600 50  0001 C CNN
+F 3 "http://datasheets.maximintegrated.com/en/ds/DS18B20.pdf" H 6000 2100 50  0001 C CNN
+	1    6150 1850
 	1    0    0    -1
 $EndComp
-Text Label 5150 2700 0    50   ~ 0
+Text Label 6800 1850 0    50   ~ 0
 P3_1
 $Comp
 L power:GND #PWR08
 U 1 1 5BE9883D
-P 4850 3000
-F 0 "#PWR08" H 4850 2750 50  0001 C CNN
-F 1 "GND" H 4855 2827 50  0000 C CNN
-F 2 "" H 4850 3000 50  0001 C CNN
-F 3 "" H 4850 3000 50  0001 C CNN
-	1    4850 3000
+P 6150 2150
+F 0 "#PWR08" H 6150 1900 50  0001 C CNN
+F 1 "GND" H 6155 1977 50  0000 C CNN
+F 2 "" H 6150 2150 50  0001 C CNN
+F 3 "" H 6150 2150 50  0001 C CNN
+	1    6150 2150
 	1    0    0    -1
 $EndComp
@@
 L power:VCC #PWR07
 U 1 1 5BE98875
-P 4850 2400
-F 0 "#PWR07" H 4850 2250 50  0001 C CNN
-F 1 "VCC" H 4867 2573 50  0000 C CNN
-F 2 "" H 4850 2400 50  0001 C CNN
-F 3 "" H 4850 2400 50  0001 C CNN
-	1    4850 2400
+P 6150 1450
+F 0 "#PWR07" H 6150 1300 50  0001 C CNN
+F 1 "VCC" H 6167 1623 50  0000 C CNN
+F 2 "" H 6150 1450 50  0001 C CNN
+F 3 "" H 6150 1450 50  0001 C CNN
+	1    6150 1450
 	1    0    0    -1
 $EndComp
@@
 Text Label 1800 2350 3    50   ~ 0
 P4_2
+Wire Wire Line
+	6450 1850 6600 1850
+Wire Wire Line
+	6600 1500 6600 1850
+Connection ~ 6600 1850
+Wire Wire Line
+	6600 1850 6800 1850
+Wire Wire Line
+	6150 1450 6150 1500
+$Comp
+L Device:R R1
+U 1 1 5BEE3DBC
+P 6350 1500
+F 0 "R1" V 6143 1500 50  0000 C CNN
+F 1 "4.7k" V 6234 1500 50  0000 C CNN
+F 2 "" V 6280 1500 50  0001 C CNN
+F 3 "~" H 6350 1500 50  0001 C CNN
+	1    6350 1500
+	0    1    1    0
+$EndComp
+Wire Wire Line
+	6150 1500 6200 1500
+Connection ~ 6150 1500
+Wire Wire Line
+	6150 1500 6150 1550
+Wire Wire Line
+	6500 1500 6600 1500
 $EndSCHEMATC
